File: FZburner-mod-toolboard.kicad_pcb (KiCad board)
At the start: 2 copper layers, 56 parts, among them J1 USB_C_Receptacle_USB2.0, Q1 FH3400C, SW1 BOOTSEL, U2 RY8310, U3 RP2040, U4 ADXL345BCCZ-RL7, U5 SHT30-DIS, U6 TMC2209, U7 LDC1612, U8 MT6131AT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

Commit message: temp commit
Parts:
- removed TP2: D-, TestPoint:TestPoint_Pad_1.5x1.5mm
- removed TP3: D+, TestPoint:TestPoint_Pad_1.5x1.5mm
- added C26: 100nF, Capacitor_SMD:C_0402_1005Metric, F.Cu at (62.5, 56.2)
- added C27: 10uF 50V, Capacitor_SMD:C_1210_3225Metric, F.Cu at (64.8, 34.0)
- added H1: MountingHole_Pad, MountingHole:MountingHole_3.2mm_M3_Pad_Via, F.Cu at (75.4, 45.7)
- added H2: MountingHole_Pad, MountingHole:MountingHole_3.2mm_M3_Pad_Via, F.Cu at (31.5, 45.7)
- added H3: MountingHole_Pad, MountingHole:MountingHole_3.2mm_M3_Pad_Via, F.Cu at (75.4, 53.2)
- added H4: MountingHole_Pad, MountingHole:MountingHole_3.2mm_M3_Pad_Via, F.Cu at (67.4, 53.2)
- added J2: Extruder_motor, Connector_JST:JST_GH_BM04B-GHS-TBT_1x04-1MP_P1.25mm_Vertical, F.Cu at (37.7, 54.3)
- added J3: hotend_connector, Library:无标题, F.Cu at (67.5, 41.9)
- added U9: W25Q16JVUXIQ, Package_SON:Winbond_USON-8-1EP_3x2mm_P0.5mm_EP0.2x1.6mm, F.Cu at (51.3, 39.1)
- Q1: value FH3400C -> WSD3050DN33
- moved R14 116.3 mm to (30.3, 50.3), turned to 180 degrees
- moved R13 113.9 mm to (30.3, 52.6), turned to 180 degrees
- moved R10 113.8 mm to (47.0, 31.4), turned to 180 degrees
- moved R9 113.1 mm to (47.0, 30.4), turned to 180 degrees
- moved R8 112.6 mm to (47.0, 29.2)
- moved R3 110.4 mm to (43.0, 33.4), turned to 90 degrees
- moved R12 110.1 mm to (34.4, 50.9), turned to -90 degrees
- moved C1 108.6 mm to (37.0, 39.2)
- moved L1 108.1 mm to (43.2, 38.3), turned to -90 degrees
- moved U2 104.4 mm to (45.7, 33.9), turned to 180 degrees
- moved U3 103.9 mm to (52.8, 45.5)
- moved U4 101.6 mm to (45.5, 43.2), turned to 90 degrees
- moved R5 101.1 mm to (54.4, 39.3), turned to -90 degrees
- moved C20 99.8 mm to (39.0, 43.7), turned to 90 degrees
- moved U8 99.8 mm to (29.6, 55.8), turned to 180 degrees
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Connections:
- C21 pad 1: Net-(U8-OUTPUT) -> X_ENDSTOP
- Q1 pad 2: unconnected-(Q1-G-Pad2) -> HEATER
- R11 pad 2: Net-(U6-ENN) -> Net-(U3-GPIO9)
- R15 pad 2: Net-(J3-Pin_4) -> Net-(J3-Pin_14)
- U3 pad 12: unconnected-(U3-GPIO9-Pad12) -> Net-(U3-GPIO9)
- U3 pad 28: unconnected-(U3-GPIO17-Pad28) -> HEATER
- U3 pad 30: unconnected-(U3-GPIO19-Pad30) -> X_ENDSTOP
- U3 pad 38: unconnected-(U3-GPIO26_ADC0-Pad38) -> Net-(J3-Pin_14)
- U3 pad 6: unconnected-(U3-GPIO4-Pad6) -> Net-(U3-GPIO4)
- U3 pad 7: unconnected-(U3-GPIO5-Pad7) -> Net-(U3-GPIO5)
- U3 pad 8: unconnected-(U3-GPIO6-Pad8) -> Net-(U3-GPIO6)
- U6 pad 14: unconnected-(U6-PDN_UART-Pad14) -> Net-(U3-GPIO4)
- U6 pad 16: unconnected-(U6-STEP-Pad16) -> Net-(U3-GPIO5)
- U6 pad 19: unconnected-(U6-DIR-Pad19) -> Net-(U3-GPIO6)
- U6 pad 2: Net-(U6-ENN) -> Net-(U3-GPIO9)
- U7 pad 11: unconnected-(U7-IN1A-Pad11) -> Net-(U7-IN1A)
- U7 pad 12: unconnected-(U7-IN1B-Pad12) -> Net-(U7-IN1B)
- U8 pad 2: Net-(U8-OUTPUT) -> X_ENDSTOP
Routing:
- net +3.3V: track 0.00 -> 82.2 mm, vias 0 -> 38
- net Net-(U3-GPIO5): track 0.00 -> 19.7 mm, vias 0 -> 2
- net Net-(U3-GPIO6): track 0.00 -> 19.7 mm, vias 0 -> 2
- net GND: track 0.00 -> 18.5 mm, vias 0 -> 95
- net Net-(U3-GPIO4): track 0.00 -> 16.8 mm, vias 0 -> 2
- net Net-(U7-IN1A): track 0.00 -> 16.1 mm
- net Net-(U3-QSPI_SS): track 0.00 -> 14.4 mm, vias 0 -> 2
- net Net-(U3-GPIO3): track 0.00 -> 12.3 mm
- net Net-(U3-GPIO9): track 0.00 -> 11.3 mm, vias 0 -> 2
- net Net-(U6-BRB): track 0.00 -> 11.1 mm
- net Net-(U3-GPIO2): track 0.00 -> 10.5 mm
- net Net-(U6-BRA): track 0.00 -> 10.2 mm
- net Net-(U3-XIN): track 0.00 -> 9.89 mm
- net Net-(U3-GPIO0): track 0.00 -> 7.34 mm
- net Net-(U7-IN1B): track 0.00 -> 7.32 mm
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- added copper zone on F.Cu, net +3.3V
- added copper zone on B.Cu, net GND
- added copper zone on F.Cu, net GND
- added copper zone on F.Cu, net Net-(J3-Pin_10)
- added copper zone on F.Cu, net Net-(U2-SW)
- added copper zone on F.Cu, net Net-(U3-VREG_VOUT)
- added copper zone on F.Cu, net VBUS
- added copper zone on In1.Cu, net VBUS
Other:
- board outline added: 52 x 36 mm
- copper layers 2 -> 4
