File: FZburner-mod-toolboard.kicad_sch (KiCad schematic)
At the start: 82 parts, among them J1 hotend_connector, J10 Probe, J2 TEMP_SENSOR, J3 X_ENDSTOP, J4 PROBE, J5 FAN1, J6 FAN2, J7 Heater, J8 Extruder_motor, J9 USB_C_Receptacle_USB2.0, Q2 FH3400C, Q3 WST4041, Q4 FH3400C, Q5 WST4041, Q6 FH3400C, Q7 WST4041, SW1 BOOTSEL, U1 W25Q16JVUXIQ, U2 RY8310, U3 RP2040, U4 TLV70233_SOT23-5, U5 ADXL345BCCZ-RL7, U6 TMC2209, U7 ??? (TO-92S), Y1 12MHz

Commit message: temp commit
Parts:
- removed C13: 47uF 16V, Capacitor_SMD:C_1210_3225Metric, symbol Device:C_Small
- removed C15: 10uF 50V, Capacitor_SMD:C_1210_3225Metric, symbol Device:C_Small
- removed H1, H2: MountingHole_Pad, MountingHole:MountingHole_3.2mm_M3_Pad_Via, symbol Mechanical:MountingHole_Pad
- removed J3: X_ENDSTOP, Connector_GH:GH_1.25_1x02_Horizontal, symbol Connector_Generic_MountingPin:Conn_01x02_MountingPin
- removed J5: FAN1, Connector_GH:GH_1.25_1x02_Horizontal, symbol Connector_Generic_MountingPin:Conn_01x02_MountingPin
- removed J6: FAN2, Connector_GH:GH_1.25_1x02_Horizontal, symbol Connector_Generic_MountingPin:Conn_01x02_MountingPin
- removed Q2, Q6: FH3400C, Package_TO_SOT_SMD:SOT-23, symbol Device:Q_NMOS_GSD
- removed Q3, Q7: WST4041, Package_TO_SOT_SMD:SOT-23, symbol Device:Q_PMOS_GSD
- removed R12, R13, R19: 10K, Resistor_SMD:R_0402_1005Metric, symbol Device:R_Small
- removed R14, R20: 1M, Resistor_SMD:R_0402_1005Metric, symbol Device:R_Small
- removed U4: TLV70233_SOT23-5, Package_TO_SOT_SMD:SOT-23-5, symbol Regulator_Linear:TLV70233_SOT23-5
- added R4: DNP, Resistor_SMD:R_0402_1005Metric, symbol Device:R_Small
- added U8: SHT30-DIS, Sensor_Humidity:Sensirion_DFN-8-1EP_2.5x2.5mm_P0.5mm_EP1.1x1.7mm, symbol Sensor_Humidity:SHT30-DIS
- R8: value 52.5K -> 10K
- R9: value 10K -> 3.2K
Connections:
- net +24V: no longer C1.1, C2.1, C9.1, R3.1, U2.5 (IN)
- net GND: now also R4.2
- net at R8.2, R9.1, U2.3 (FB): now also R4.1
- net at J2.1 (Pin_1), R11.2: no longer U3.38 (GPIO26_ADC0)
- net at Q4.1 (G), R18.1: no longer U3.12 (GPIO9)
- net at J4.1 (Pin_1), R16.2: no longer U3.27 (GPIO16)
- net at R15.2, U6.2 (ENN): no longer U3.28 (GPIO17)
- net at U3.36 (GPIO24): no longer U6.19 (DIR)
- net at U3.37 (GPIO25): no longer U6.16 (STEP)
- net at U3.41 (GPIO29_ADC3): no longer U6.14 (PDN_UART)
- net VBUS: now reaches J9.A4 (VBUS), J9.A9 (VBUS), J9.B4 (VBUS), J9.B9 (VBUS)
- net VBUS: now also C1.1, C2.1, C9.1, R3.1, U2.5 (IN)
- new net: U8.8 (VSS), U8.9 (VSS)
- no-connect marks 9 -> 10
Other:
- note removed: "Add 5V/24V switch here"
- moved on the sheet: C1, C10, C11, C12, C14, C16, C17, C18, C19, C2, C20, C21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

Commit message: temp_commit
Parts:
- removed C17: 100nF, symbol Device:C_Small
- removed C19: 10uF 50V, Capacitor_SMD:C_1210_3225Metric, symbol Device:C_Small
- removed D1: GREEN, symbol Device:LED_Small
- removed J10: Probe, symbol Connector_Generic_MountingPin:Conn_01x04_MountingPin
- removed J2: TEMP_SENSOR, Connector_GH:GH_1.25_1x02_Horizontal, symbol Connector_Generic_MountingPin:Conn_01x02_MountingPin
- removed J4: PROBE, Connector_GH:GH_1.25_1x02_Horizontal, symbol Connector_Generic_MountingPin:Conn_01x02_MountingPin
- removed J7: Heater, TerminalBlock_TE-Connectivity:TerminalBlock_TE_282834-2_1x02_P2.54mm_Horizontal, symbol Connector_Generic:Conn_01x02
- removed Q4: FH3400C, Package_TO_SOT_SMD:SOT-23, symbol Device:Q_NMOS_GSD
- removed Q5: WST4041, Package_TO_SOT_SMD:SOT-23, symbol Device:Q_PMOS_GSD
- removed R1: 1K, symbol Device:R_Small
- removed R10: 10K, symbol Device:R_Small
- removed R11: 4.7K, Resistor_SMD:R_0402_1005Metric, symbol Device:R_Small
- removed R16, R17: 10K, Resistor_SMD:R_0402_1005Metric, symbol Device:R_Small
- removed R18: 1M, Resistor_SMD:R_0402_1005Metric, symbol Device:R_Small
- removed TP4, TP5: MAG, symbol Connector:TestPoint_Small
- removed U7: ??? (TO-92S), Package_TO_SOT_THT:TO-92S, symbol Sensor_Magnetic:DRV5033FAxLPG
- added C21, C23: 1nF, Capacitor_SMD:C_0402_1005Metric, symbol Device:C_Small
- added C22, C24, C25: 100nF, Capacitor_SMD:C_0402_1005Metric, symbol Device:C_Small
- added Q1: FH3400C, Package_TO_SOT_SMD:SOT-23, symbol Transistor_FET:Q_NMOS_DGS
- added R15: 4.7K, Resistor_SMD:R_0402_1005Metric, symbol Device:R_Small
- added U7: LDC1612, Package_SON:WSON-12-1EP_4x4mm_P0.5mm_EP2.6x3mm_ThermalVias, symbol Sensor_Proximity:LDC1612
- added U8: MT6131AT, Package_TO_SOT_SMD:SOT-23, symbol Sensor_Magnetic:SM351LT
- added Y2: OT2EL4C4JI-111OLP-40M, Crystal:Crystal_SMD_3225-4Pin_3.2x2.5mm, symbol Oscillator:ASCO
- renumbered C7 to C10, C10 to C11, C11 to C12, C12 to C13, C18 to C15, C20 to C16, C21 to C17, C22 to C18, C23 to C19, C24 to C20, C9 to C4, C4 to C5, C5 to C7, C16 to C8, C8 to C9, J9 to J1, J8 to J2, J1 to J3, R2 to R1, R4 to R10, R15 to R11, R23 to R12, R21 to R13, R22 to R14, R24 to R2, R5 to R4, R6 to R5, R25 to R6, TP3 to TP1, TP1 to TP2, TP2 to TP3, U5 to U4, U8 to U5
Connections:
- net +24V is gone; now on net VBUS: C15.1, C16.1, U6.22 (VS), U6.28 (VS)
- net +3V3 is gone; now on net +3.3V: C11.1, C12.1, C13.1, C14.1, C17.1, C18.1, C3.1, R11.1, R7.1, U1.8 (VCC), U3.1 (IOVDD), U3.10 (IOVDD), U3.22 (IOVDD), U3.33 (IOVDD), U3.42 (IOVDD), U3.43 (ADC_AVDD), U3.44 (VREG_IN), U3.48 (USB_VDD), U3.49 (IOVDD), U4.1 (Vdd_I/O), U4.3 (RES), U4.6 (Vs), U6.15 (VCC_IO)
- net +3.3V: now also C10.1, L1.2, R8.1, C22.1, C23.1, C24.1, C25.1, R15.1, U7.7 (VDD), U8.1 (VCC), Y2.4 (VDD)
- net GND: now also J3.6 (Pin_6), J3.7 (Pin_7), C21.2, C22.2, C23.2, C24.2, C25.2, Q1.3 (S), U7.13 (GND), U7.8 (GND), U8.3 (GND), Y2.1 (Tri-State), Y2.2 (GND)
- net VBUS: now also J3.1 (Pin_1), J3.2 (Pin_2), J3.3 (Pin_3)
- net at J3.10 (Pin_10), J3.8 (Pin_8), J3.9 (Pin_9): now also Q1.1 (D)
- net at J3.4 (Pin_4), J3.5 (Pin_5): now also R15.2
- new net: U7.3 (CLKIN), Y2.3 (OUT)
- new net: C21.1, U8.2 (OUTPUT)
Other:
- note removed: "Endstop & Probe"
- note removed: "NTC+"
- note removed: "NTC-"
- note removed: "P+"
- note removed: "P-"
- note removed: "√step driver √fan1 √fan2 √x_endstop √probe √heater √temp_sensor"
- moved on the sheet: J3, U5

Commit message: temp commit
Parts:
- removed TP2: D-, TestPoint:TestPoint_Pad_1.5x1.5mm, symbol Connector:TestPoint
- removed TP3: D+, TestPoint:TestPoint_Pad_1.5x1.5mm, symbol Connector:TestPoint
- removed U1: W25Q16JVUXIQ, Package_SON:USON-8_3.0x2.0mm_P0.5mm, symbol Memory_Flash:W25Q32JVSS
- added C26: 100nF, Capacitor_SMD:C_0402_1005Metric, symbol Device:C_Small
- added C27: 10uF 50V, Capacitor_SMD:C_1210_3225Metric, symbol Device:C_Small
- added H1, H2, H3, H4: MountingHole_Pad, MountingHole:MountingHole_3.2mm_M3_Pad_Via, symbol Mechanical:MountingHole_Pad
- added U9: W25Q16JVUXIQ, Package_SON:Winbond_USON-8-1EP_3x2mm_P0.5mm_EP0.2x1.6mm, symbol Memory_RAM:APS1604M-3SQRx-ZR
- J2: footprint Connector_GH:GH_1.25_1x04_Veritical -> Connector_JST:JST_GH_BM04B-GHS-TBT_1x04-1MP_P1.25mm_Vertical
- J3: footprint (none) -> Library:无标题
- Q1: value FH3400C -> WSD3050DN33
Connections:
- net +3.3V: now also U9.8 (VDD)
- net GND: now also J3.16 (Pin_16), J3.17 (Pin_17), C27.2, H1.1, H2.1, U9.4 (VSS), U9.9 (EPAD)
- net VBUS: now also J3.11 (Pin_11), J3.12 (Pin_12), J3.13 (Pin_13), C27.1
- net at R2.1, U3.56 (QSPI_SS): now also U9.1 (~{CE})
- net at U7.11 (IN1A): now also C26.1, H3.1
- net at U7.12 (IN1B): now also C26.2, H4.1
- net at U3.12 (GPIO9): now also R11.2, U6.2 (ENN)
- net HEATER: now reaches U3.28 (GPIO17)
- net HEATER: now also Q1.2 (G)
- net X_ENDSTOP: now reaches U3.30 (GPIO19)
- net X_ENDSTOP: now also C21.1, U8.2 (OUTPUT)
- net at U3.38 (GPIO26_ADC0): now also J3.14 (Pin_14), J3.15 (Pin_15), J3.4 (Pin_4), J3.5 (Pin_5), R15.2
- net at U3.51 (QSPI_SD3): now also U9.7 (SIO3)
- net at U3.52 (QSPI_SCLK): now also U9.6 (SCLK)
- net at U3.53 (QSPI_SD0): now also U9.5 (SI/SIO0)
- net at U3.54 (QSPI_SD2): now also U9.3 (SIO2)
- net at U3.55 (QSPI_SD1): now also U9.2 (SO/SIO1)
- net at U3.6 (GPIO4): now also U6.14 (PDN_UART)
- net at U3.7 (GPIO5): now also U6.16 (STEP)
- net at U3.8 (GPIO6): now also U6.19 (DIR)
- net at J3.10 (Pin_10), J3.8 (Pin_8), J3.9 (Pin_9)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: now also J3.18 (Pin_18), J3.19 (Pin_19), J3.20 (Pin_20)
- net at J2.1 (Pin_1): now also U6.1 (OB2); no longer U6.21 (OA2)
- net at J2.2 (Pin_2): now also U6.26 (OB1); no longer U6.24 (OA1)
- net at J2.3 (Pin_3): now also U6.24 (OA1); no longer U6.26 (OB1)
- net at J2.4 (Pin_4): now also U6.21 (OA2); no longer U6.1 (OB2)
Other:
- moved on the sheet: C21, C22, C23, C24, C25, J3, Q1, R15, U5, U7, U8, Y2
